Commit message: Add files via upload

File: src/allegro_hand_controllers/urdf/allegro_hand_description_left_A.urdf (robot description, URDF)
Before this commit: robot allegro_hand_left, 22 links, 21 joints
Links:
- link link_0_0: geometry collision mesh filename=package://allegro_hand_controllers/meshes/l1.stl scale=0.001 0.001 0.001; visual mesh filename=package://allegro_hand_controllers/meshes/l1.stl scale=0.001 0.001 0.001
- link link_10_0: geometry collision mesh filename=package://allegro_hand_controllers/meshes/l3.stl scale=0.001 0.001 0.001; visual mesh filename=package://allegro_hand_controllers/meshes/l3.stl scale=0.001 0.001 0.001
- link link_11_0: geometry collision mesh filename=package://allegro_hand_controllers/meshes/l4.stl scale=0.001 0.001 0.001; visual mesh filename=package://allegro_hand_controllers/meshes/l4.stl scale=0.001 0.001 0.001
- link link_11_0_tip: geometry collision mesh filename=package://allegro_hand_controllers/meshes/finger_tip.stl scale=0.001 0.001 0.001; visual mesh filename=package://allegro_hand_controllers/meshes/finger_tip.stl scale=0.001 0.001 0.001
- link link_12_0: geometry collision mesh filename=package://allegro_hand_controllers/meshes/t1_set.stl scale=0.001 0.001 0.001; visual mesh filename=package://allegro_hand_controllers/meshes/t1_set.stl scale=0.001 0.001 0.001
- link link_13_0: geometry collision mesh filename=package://allegro_hand_controllers/meshes/t2_set.stl scale=0.001 0.001 0.001; visual mesh filename=package://allegro_hand_controllers/meshes/t2_set.stl scale=0.001 0.001 0.001
- link link_14_0: geometry collision mesh filename=package://allegro_hand_controllers/meshes/t3_set.stl scale=0.001 0.001 0.001; visual mesh filename=package://allegro_hand_controllers/meshes/t3_set.stl scale=0.001 0.001 0.001
- link link_15_0: geometry collision mesh filename=package://allegro_hand_controllers/meshes/t4_set.stl scale=0.001 0.001 0.001; visual mesh filename=package://allegro_hand_controllers/meshes/t4_set.stl scale=0.001 0.001 0.001
- link link_15_0_tip: geometry collision mesh filename=package://allegro_hand_controllers/meshes/finger_tip_silico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 scale=0.001 0.001 0.001; visual mesh filename=package://allegro_hand_controllers/meshes/finger_tip_silico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 scale=0.001 0.001 0.001
- link link_1_0: geometry collision mesh filename=package://allegro_hand_controllers/meshes/l2.stl scale=0.001 0.001 0.001; visual mesh filename=package://allegro_hand_controllers/meshes/l2.stl scale=0.001 0.001 0.001
- link link_2_0: geometry collision mesh filename=package://allegro_hand_controllers/meshes/l3.stl scale=0.001 0.001 0.001; visual mesh filename=package://allegro_hand_controllers/meshes/l3.stl scale=0.001 0.001 0.001
- link link_3_0: geometry collision mesh filename=package://allegro_hand_controllers/meshes/l4.stl scale=0.001 0.001 0.001; visual mesh filename=package://allegro_hand_controllers/meshes/l4.stl scale=0.001 0.001 0.001
- link link_3_0_tip: geometry collision mesh filename=package://allegro_hand_controllers/meshes/finger_tip.stl scale=0.001 0.001 0.001; visual mesh filename=package://allegro_hand_controllers/meshes/finger_tip.stl scale=0.001 0.001 0.001
- link link_4_0: geometry collision mesh filename=package://allegro_hand_controllers/meshes/l1.stl scale=0.001 0.001 0.001; visual mesh filename=package://allegro_hand_controllers/meshes/l1.stl scale=0.001 0.001 0.001
- link link_5_0: geometry collision mesh filename=package://allegro_hand_controllers/meshes/l2.stl scale=0.001 0.001 0.001; visual mesh filename=package://allegro_hand_controllers/meshes/l2.stl scale=0.001 0.001 0.001
- link link_6_0: geometry collision mesh filename=package://allegro_hand_controllers/meshes/l3.stl scale=0.001 0.001 0.001; visual mesh filename=package://allegro_hand_controllers/meshes/l3.stl scale=0.001 0.001 0.001
- link link_7_0: geometry collision mesh filename=package://allegro_hand_controllers/meshes/l4.stl scale=0.001 0.001 0.001; visual mesh filename=package://allegro_hand_controllers/meshes/l4.stl scale=0.001 0.001 0.001
- link link_7_0_tip: geometry collision mesh filename=package://allegro_hand_controllers/meshes/finger_tip.stl scale=0.001 0.001 0.001; visual mesh filename=package://allegro_hand_controllers/meshes/finger_tip.stl scale=0.001 0.001 0.001
- link link_8_0: geometry collision mesh filename=package://allegro_hand_controllers/meshes/l1.stl scale=0.001 0.001 0.001; visual mesh filename=package://allegro_hand_controllers/meshes/l1.stl scale=0.001 0.001 0.001
- link link_9_0: geometry collision mesh filename=package://allegro_hand_controllers/meshes/l2.stl scale=0.001 0.001 0.001; visual mesh filename=package://allegro_hand_controllers/meshes/l2.stl scale=0.001 0.001 0.001
- link palm_link: geometry collision mesh filename=package://allegro_hand_controllers/meshes/left_hand_G.stl scale=0.001 0.001 0.001; visual mesh filename=package://allegro_hand_controllers/meshes/left_hand_G.stl scale=0.001 0.001 0.001

File: src/allegro_hand_controllers/urdf/allegro_hand_description_right_A.urdf (robot description, URDF)
Before this commit: robot allegro_hand_right, 22 links, 21 joints
Links:
- link link_0_0: geometry collision mesh filename=package://allegro_hand_controllers/meshes/l1.stl scale=0.001 0.001 0.001; visual mesh filename=package://allegro_hand_controllers/meshes/l1.stl scale=0.001 0.001 0.001
- link link_10_0: geometry collision mesh filename=package://allegro_hand_controllers/meshes/l3.stl scale=0.001 0.001 0.001; visual mesh filename=package://allegro_hand_controllers/meshes/l3.stl scale=0.001 0.001 0.001
- link link_11_0: geometry collision mesh filename=package://allegro_hand_controllers/meshes/l4.stl scale=0.001 0.001 0.001; visual mesh filename=package://allegro_hand_controllers/meshes/l4.stl scale=0.001 0.001 0.001
- link link_11_0_tip: geometry collision mesh filename=package://allegro_hand_controllers/meshes/finger_tip.stl scale=0.001 0.001 0.001; visual mesh filename=package://allegro_hand_controllers/meshes/finger_tip.stl scale=0.001 0.001 0.001
- link link_12_0: geometry collision mesh filename=package://allegro_hand_controllers/meshes/t1_set.stl scale=0.001 0.001 0.001; visual mesh filename=package://allegro_hand_controllers/meshes/t1_set.stl scale=0.001 0.001 0.001
- link link_13_0: geometry collision mesh filename=package://allegro_hand_controllers/meshes/t2_set.stl scale=0.001 0.001 0.001; visual mesh filename=package://allegro_hand_controllers/meshes/t2_set.stl scale=0.001 0.001 0.001
- link link_14_0: geometry collision mesh filename=package://allegro_hand_controllers/meshes/t3_set.stl scale=0.001 0.001 0.001; visual mesh filename=package://allegro_hand_controllers/meshes/t3_set.stl scale=0.001 0.001 0.001
- link link_15_0: geometry collision mesh filename=package://allegro_hand_controllers/meshes/t4_set.stl scale=0.001 0.001 0.001; visual mesh filename=package://allegro_hand_controllers/meshes/t4_set.stl scale=0.001 0.001 0.001
- link link_15_0_tip: geometry collision mesh filename=package://allegro_hand_controllers/meshes/finger_tip_silico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 scale=0.001 0.001 0.001; visual mesh filename=package://allegro_hand_controllers/meshes/finger_tip_silico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 scale=0.001 0.001 0.001
- link link_1_0: geometry collision mesh filename=package://allegro_hand_controllers/meshes/l2.stl scale=0.001 0.001 0.001; visual mesh filename=package://allegro_hand_controllers/meshes/l2.stl scale=0.001 0.001 0.001
- link link_2_0: geometry collision mesh filename=package://allegro_hand_controllers/meshes/l3.stl scale=0.001 0.001 0.001; visual mesh filename=package://allegro_hand_controllers/meshes/l3.stl scale=0.001 0.001 0.001
- link link_3_0: geometry collision mesh filename=package://allegro_hand_controllers/meshes/l4.stl scale=0.001 0.001 0.001; visual mesh filename=package://allegro_hand_controllers/meshes/l4.stl scale=0.001 0.001 0.001
- link link_3_0_tip: geometry collision mesh filename=package://allegro_hand_controllers/meshes/finger_tip.stl scale=0.001 0.001 0.001; visual mesh filename=package://allegro_hand_controllers/meshes/finger_tip.stl scale=0.001 0.001 0.001
- link link_4_0: geometry collision mesh filename=package://allegro_hand_controllers/meshes/l1.stl scale=0.001 0.001 0.001; visual mesh filename=package://allegro_hand_controllers/meshes/l1.stl scale=0.001 0.001 0.001
- link link_5_0: geometry collision mesh filename=package://allegro_hand_controllers/meshes/l2.stl scale=0.001 0.001 0.001; visual mesh filename=package://allegro_hand_controllers/meshes/l2.stl scale=0.001 0.001 0.001
- link link_6_0: geometry collision mesh filename=package://allegro_hand_controllers/meshes/l3.stl scale=0.001 0.001 0.001; visual mesh filename=package://allegro_hand_controllers/meshes/l3.stl scale=0.001 0.001 0.001
- link link_7_0: geometry collision mesh filename=package://allegro_hand_controllers/meshes/l4.stl scale=0.001 0.001 0.001; visual mesh filename=package://allegro_hand_controllers/meshes/l4.stl scale=0.001 0.001 0.001
- link link_7_0_tip: geometry collision mesh filename=package://allegro_hand_controllers/meshes/finger_tip.stl scale=0.001 0.001 0.001; visual mesh filename=package://allegro_hand_controllers/meshes/finger_tip.stl scale=0.001 0.001 0.001
- link link_8_0: geometry collision mesh filename=package://allegro_hand_controllers/meshes/l1.stl scale=0.001 0.001 0.001; visual mesh filename=package://allegro_hand_controllers/meshes/l1.stl scale=0.001 0.001 0.001
- link link_9_0: geometry collision mesh filename=package://allegro_hand_controllers/meshes/l2.stl scale=0.001 0.001 0.001; visual mesh filename=package://allegro_hand_controllers/meshes/l2.stl scale=0.001 0.001 0.001
- link palm_link: geometry collision mesh filename=package://allegro_hand_controllers/meshes/palm.stl scale=0.001 0.001 0.001; visual mesh filename=package://allegro_hand_controllers/meshes/palm.stl scale=0.001 0.001 0.001

Commit message: Add files via upload

File: src/allegro_hand_controllers/urdf/allegro_hand_description_left_A.urdf (robot description, URDF)
Before this commit: robot allegro_hand_left, 22 links, 21 joints
Links:
- link link_0_0: mass 0.0119 -> 0.0176
- link link_10_0: mass 0.0355 -> 0.0366
- link link_11_0: mass 0.0096 -> 0.00569
- link link_11_0_tip: mass 0.0168 -> 0.00
- link link_1_0: mass 0.065 -> 0.066
- link link_2_0: mass 0.0355 -> 0.0366
- link link_3_0: mass 0.0096 -> 0.00569
- link link_3_0_tip: mass 0.0168 -> 0.00
- link link_4_0: mass 0.0119 -> 0.0176
- link link_5_0: mass 0.065 -> 0.066
- link link_6_0: mass 0.0355 -> 0.0366
- link link_7_0: mass 0.0096 -> 0.00569
- link link_7_0_tip: mass 0.0168 -> 0.00
- link link_8_0: mass 0.0119 -> 0.0176
- link link_9_0: mass 0.065 -> 0.066
Joints:
- joint joint_10_0: limit lower=-0.174 upper=1.709 effort=15 velocity=7 -> lower=-0.174 upper=1.9 effort=15 velocity=7
- joint joint_11_0: limit lower=-0.227 upper=1.618 effort=15 velocity=7 -> lower=-0.227 upper=1.9 effort=15 velocity=7
- joint joint_12_0: limit lower=-1.78 upper=0.00 effort=15 velocity=7 -> lower=-1.78 upper=0.5 effort=15 velocity=7
- joint joint_13_0: limit lower=1.4 upper=3.22 effort=15 velocity=7 -> lower=1.0 upper=3.22 effort=15 velocity=7
- joint joint_14_0: limit lower=-1.85 upper=0.05 effort=15 velocity=7 -> lower=-1.85 upper=0.2 effort=15 velocity=7
- joint joint_15_0: limit lower=-1.80 upper=0.09 effort=15 velocity=7 -> lower=-1.80 upper=0.2 effort=15 velocity=7
- joint joint_1_0: limit lower=-0.196 upper=1.61 effort=15 velocity=7 -> lower=-0.196 upper=1.9 effort=15 velocity=7
- joint joint_2_0: limit lower=-0.174 upper=1.709 effort=15 velocity=7 -> lower=-0.174 upper=1.9 effort=15 velocity=7
- joint joint_3_0: limit lower=-0.227 upper=1.618 effort=15 velocity=7 -> lower=-0.227 upper=1.9 effort=15 velocity=7
- joint joint_5_0: limit lower=-0.196 upper=1.61 effort=15 velocity=7 -> lower=-0.196 upper=1.9 effort=15 velocity=7
- joint joint_6_0: limit lower=-0.174 upper=1.709 effort=15 velocity=7 -> lower=-0.174 upper=1.9 effort=15 velocity=7
- joint joint_7_0: limit lower=-0.227 upper=1.618 effort=15 velocity=7 -> lower=-0.227 upper=1.9 effort=15 velocity=7
- joint joint_9_0: limit lower=-0.196 upper=1.61 effort=15 velocity=7 -> lower=-0.196 upper=1.9 effort=15 velocity=7

File: src/allegro_hand_controllers/urdf/allegro_hand_description_right_A.urdf (robot description, URDF)
Before this commit: robot allegro_hand_right, 22 links, 21 joints
Links:
- link link_0_0: mass 0.0119 -> 0.0176
- link link_10_0: mass 0.0355 -> 0.0366
- link link_11_0: mass 0.0096 -> 0.00569
- link link_11_0_tip: mass 0.0168 -> 0.00
- link link_15_0: mass 0.0334 -> 0.0338
- link link_15_0_tip: mass 0.0014 -> 0.00
- link link_1_0: mass 0.065 -> 0.066
- link link_2_0: mass 0.0355 -> 0.0366
- link link_3_0: mass 0.0096 -> 0.00569
- link link_3_0_tip: mass 0.0168 -> 0.00
- link link_4_0: mass 0.0119 -> 0.0176
- link link_5_0: mass 0.065 -> 0.066
- link link_6_0: mass 0.0355 -> 0.0366
- link link_7_0: mass 0.0096 -> 0.00569
- link link_7_0_tip: mass 0.0168 -> 0.00
- link link_8_0: mass 0.0119 -> 0.0176
- link link_9_0: mass 0.065 -> 0.066
